Commit message: ADD Particle concentration sensor to robot description
Signed-off-by: Musa Morena Marcusso Manhaes <Musa.Marcusso@de.bosch.com>

File: desistek_saga_description/urdf/desistek_saga_sensors.xacro (robot description, xacro)
@@ -29,5 +29,5 @@
       <origin xyz="0.2 0 0.0" rpy="0 0 0"/>
   </xacro:regular_camera_plugin_macro>
-  <!-- Mount a 3D pose sensor -->
+  <!-- Add a 3D pose sensor -->
   <gazebo>
     <plugin name="pose_3d_plugin" filename="libgazebo_ros_p3d.so">
@@ -44,5 +44,9 @@
     <origin xyz="0.0 0 -0.1" rpy="0 0 0"/>
   </xacro:forward_multibeam_p900>
-  <!-- Mount a GPS. -->
+  <!-- Add a GPS. -->
   <xacro:default_gps namespace="${namespace}" parent_link="${namespace}/base_link" />
+  <!-- Add a chemical particle concentration sensor -->
+  <xacro:default_chemical_concentration_sensor namespace="${namespace}" parent_link="${namespace}/base_link">
+    <origin xyz="0 0 0" rpy="0 0 0"/>
+  </xacro:default_chemical_concentration_sensor>
 </robot>

Commit message: UPDATE Sensor plugin macros to use inertial_reference_frame argument
Signed-off-by: Musa Morena Marcusso Manhaes <Musa.Marcusso@de.bosch.com>

File: desistek_saga_description/urdf/desistek_saga_sensors.xacro (robot description, xacro)
@@ -29,21 +29,22 @@
       <origin xyz="0.2 0 0.0" rpy="0 0 0"/>
   </xacro:regular_camera_plugin_macro>
-  <!-- Add a 3D pose sensor -->
-  <gazebo>
-    <plugin name="pose_3d_plugin" filename="libgazebo_ros_p3d.so">
-      <robotNamespace>${namespace}</robotNamespace>
-      <bodyName>${namespace}/base_link</bodyName>
-      <topicName>pose_gt</topicName>
-      <frameName>world</frameName>
-      <gaussianNoise>0.0</gaussianNoise>
-      <updateRate>30</updateRate>
-    </plugin>
-  </gazebo>
+  <!-- Mount a GPS. -->
+  <xacro:default_gps namespace="${namespace}" parent_link="${namespace}/base_link" />
+  <!-- Mount a Pose 3D sensor. -->
+  <xacro:default_pose_3d_macro
+    namespace="${namespace}"
+    parent_link="${namespace}/base_link"
+    inertial_reference_frame="${inertial_reference_frame}" />
   <!-- Forward-looking sonar sensor -->
   <xacro:forward_multibeam_p900 namespace="${namespace}" parent_link="${namespace}/base_link">
     <origin xyz="0.0 0 -0.1" rpy="0 0 0"/>
   </xacro:forward_multibeam_p900>
-  <!-- Add a GPS. -->
-  <xacro:default_gps namespace="${namespace}" parent_link="${namespace}/base_link" />
+  <!-- IMU  -->
+  <xacro:default_imu_macro
+    namespace="${namespace}"
+    parent_link="${namespace}/base_link"
+    inertial_reference_frame="${inertial_reference_frame}">
+    <origin xyz="0 0 0" rpy="0 0 0"/>
+  </xacro:default_imu_macro>
   <!-- Add a chemical particle concentration sensor -->
   <xacro:default_chemical_concentration_sensor namespace="${namespace}" parent_link="${namespace}/base_link">
