Commit message: FIX Path to XACRO dependencies after refactoring
Signed-off-by: Musa Morena Marcusso Manhaes <musa.marcusso@de.bosch.com>

File: desistek_saga_description/urdf/desistek_saga_base.urdf.xacro (robot description, xacro)
@@ -13,5 +13,5 @@
 -->
 <robot xmlns:xacro="http://www.ros.org/wiki/xacro">
-  <xacro:include filename="$(find uuv_descriptions)/models/common/urdf/common.urdf.xacro"/>
+  <xacro:include filename="$(find uuv_descriptions)/urdf/common.urdf.xacro"/>
   <xacro:include filename="$(find uuv_sensor_ros_plugins)/urdf/sensor_snippets.xacro"/>
   <xacro:include filename="$(find desistek_saga_description)/urdf/desistek_saga_snippets.xacro"/>
@@ -28,6 +28,6 @@
   <xacro:property name="z_size" value="0.28066"/>
   <xacro:property name="equivalent_radius" value="${0.5*z_size}"/>
-  <xacro:property name="visual_mesh_file" value="file://$(find desistek_saga_description)/mesh/saga.dae"/>
-  <xacro:property name="collision_mesh_file" value="file://$(find desistek_saga_description)/mesh/saga.stl"/>
+  <xacro:property name="visual_mesh_file" value="file://$(find desistek_saga_description)/meshes/saga.dae"/>
+  <xacro:property name="collision_mesh_file" value="file://$(find desistek_saga_description)/meshes/saga.stl"/>
   <xacro:macro name="desistek_saga_base" params="namespace debug inertial_reference_frame">
   <link name="${namespace}/base_link">
@@ -57,5 +57,5 @@
     <!-- Set up hydrodynamic plugin -->
     <gazebo>
-      <plugin name="${namespace}_uuv_plugin" filename="libunderwater_object_ros_plugin.so">
+      <plugin name="${namespace}_uuv_plugin" filename="libuuv_underwater_object_ros_plugin.so">
         <fluid_density>${rho}</fluid_density>
         <flow_velocity_topic>hydrodynamics/current_velocity</flow_velocity_topic>

File: desistek_saga_description/urdf/desistek_saga_snippets.xacro (robot description, xacro)
@@ -13,5 +13,5 @@
 -->
 <robot xmlns:xacro="http://www.ros.org/wiki/xacro">
-  <xacro:property name="prop_mesh_file" value="file://$(find desistek_saga_description)/mesh/propeller.dae"/>
+  <xacro:property name="prop_mesh_file" value="file://$(find desistek_saga_description)/meshes/propeller.dae"/>
   <!-- Thruster macro with integration of joint and link-->
   <xacro:macro name="thruster_macro" params="robot_namespace thruster_id *origin">
@@ -37,5 +37,5 @@
     </joint>
     <gazebo>
-      <plugin name="${robot_namespace}_${thruster_id}_thruster_model" filename="libthruster_ros_plugin.so">
+      <plugin name="${robot_namespace}_${thruster_id}_thruster_model" filename="libuuvthruster_ros_plugin.so">
         <linkName>${robot_namespace}/thruster_${thruster_id}</linkName>
         <jointName>${robot_namespace}/thruster_${thruster_id}_joint</jointName>
