Commit message: Fix thruster macro
Signed-off-by: Musa Morena Marcusso Manhaes <Musa.Marcusso@de.bosch.com>

File: desistek_saga_description/urdf/desistek_saga_snippets.xacro (robot description, xacro)
@@ -15,5 +15,5 @@
   <xacro:property name="prop_mesh_file" value="file://$(find desistek_saga_description)/mesh/propeller.dae"/>
   <!-- Thruster macro with integration of joint and link-->
-  <xacro:macro name="thruster_macro" params="robot_namespace thruster_id *origin">
+  <!-- <xacro:macro name="thruster_macro" params="robot_namespace thruster_id *origin">
     <link name="${robot_namespace}/thruster_${thruster_id}">
       <visual>
@@ -37,5 +37,5 @@
     </joint>
     <gazebo>
-      <plugin name="${robot_namespace}_${thruster_id}_thruster_model" filename="libthruster_ros_plugin.so">
+      <plugin name="${robot_namespace}_${thruster_id}_thruster_model" filename="libuuv_thruster_ros_plugin.so">
         <linkName>${robot_namespace}/thruster_${thruster_id}</linkName>
         <jointName>${robot_namespace}/thruster_${thruster_id}_joint</jointName>
@@ -55,4 +55,16 @@
       <selfCollide>false</selfCollide>
     </gazebo>
+  </xacro:macro> -->
+  <!-- Thruster joint and link snippet -->
+  <xacro:macro name="thruster_macro"
+    params="robot_namespace thruster_id *origin">
+    <xacro:thruster_module_first_order_basic_fcn_macro
+      namespace="${robot_namespace}"
+      thruster_id="${thruster_id}"
+      mesh_filename="${prop_mesh_file}"
+      dyn_time_constant="0.05"
+      rotor_constant="0.00001">
+      <xacro:insert_block name="origin"/>
+    </xacro:thruster_module_first_order_basic_fcn_macro>
   </xacro:macro>
 </robot>

Commit message: Replace thruster macro to default snippet
Signed-off-by: Musa Morena Marcusso Manhaes <Musa.Marcusso@de.bosch.com>

File: desistek_saga_description/urdf/desistek_saga_snippets.xacro (robot description, xacro)
@@ -14,46 +14,4 @@
 <robot xmlns:xacro="http://www.ros.org/wiki/xacro">
   <xacro:property name="prop_mesh_file" value="file://$(find desistek_saga_description)/mesh/propeller.dae"/>
-  <!-- Thruster macro with integration of joint and link-->
-  <!-- <xacro:macro name="thruster_macro" params="robot_namespace thruster_id *origin">
-    <link name="${robot_namespace}/thruster_${thruster_id}">
-      <visual>
-        <geometry>
-          <mesh filename="${prop_mesh_file}" scale="1 1 1" />
-        </geometry>
-      </visual>
-      <inertial>
-        <mass value="0.001" />
-        <origin xyz="0 0 0" rpy="0 0 0"/>
-        <inertia ixx="0.000000017" ixy="0.0" ixz="0.0"
-               iyy="0.000000017" iyz="0.0"
-               izz="0.000000017" />
-      </inertial>
-    </link>
-    <joint name="${robot_namespace}/thruster_${thruster_id}_joint" type="continuous">
-      <xacro:insert_block name="origin" />
-      <axis xyz="1 0 0" />
-      <parent link="${robot_namespace}/base_link" />
-      <child link="${robot_namespace}/thruster_${thruster_id}" />
-    </joint>
-    <gazebo>
-      <plugin name="${robot_namespace}_${thruster_id}_thruster_model" filename="libuuv_thruster_ros_plugin.so">
-        <linkName>${robot_namespace}/thruster_${thruster_id}</linkName>
-        <jointName>${robot_namespace}/thruster_${thruster_id}_joint</jointName>
-        <thrusterID>${thruster_id}</thrusterID>
-        <gain>5</gain>
-        <dynamics>
-          <type>FirstOrder</type>
-          <timeConstant>0.2</timeConstant>
-        </dynamics>
-        <conversion>
-          <type>Basic</type>
-          <rotorConstant>0.00001</rotorConstant>
-        </conversion>
-      </plugin>
-    </gazebo>
-    <gazebo reference="${robot_namespace}/thruster_${thruster_id}">
-      <selfCollide>false</selfCollide>
-    </gazebo>
-  </xacro:macro> -->
   <!-- Thruster joint and link snippet -->
   <xacro:macro name="thruster_macro"
