Commit message: ADD inertial_reference_frame input argument in XACRO files
Signed-off-by: Musa Morena Marcusso Manhaes <Musa.Marcusso@de.bosch.com>

File: desistek_saga_description/robots/desistek_saga_default.xacro (robot description, xacro)
@@ -15,14 +15,13 @@
   <xacro:arg name="debug" default="0"/>
   <xacro:arg name="namespace" default="desistek_saga"/>
+  <xacro:arg name="inertial_reference_frame" default="world"/>
   <!-- Include the ROV macro file -->
   <xacro:include filename="$(find desistek_saga_description)/urdf/desistek_saga_base.urdf.xacro"/>
   <!-- Create the desistek_saga -->
-  <xacro:desistek_saga_base namespace="$(arg namespace)" debug="$(arg debug)"/>
-  <!-- Joint state publisher plugin -->
-  <gazebo>
-    <plugin name="joint_state_publisher" filename="libjoint_state_publisher.so">
-      <robotNamespace>$(arg namespace)</robotNamespace>
-      <updateRate>50</updateRate>
-    </plugin>
-  </gazebo>
+  <xacro:desistek_saga_base
+    namespace="$(arg namespace)"
+    debug="$(arg debug)"
+    inertial_reference_frame="$(arg inertial_reference_frame)"/>
+    <!-- Joint state publisher plugin -->
+    <xacro:default_joint_state_publisher namespace="$(arg namespace)" update_rate="5"/>
 </robot>

File: desistek_saga_description/urdf/desistek_saga_base.urdf.xacro (robot description, xacro)
@@ -16,4 +16,5 @@
   <xacro:include filename="$(find uuv_sensor_ros_plugins)/urdf/sensor_snippets.xacro"/>
   <xacro:include filename="$(find desistek_saga_description)/urdf/desistek_saga_snippets.xacro"/>
+  <xacro:include filename="$(find uuv_gazebo_ros_plugins)/urdf/snippets.xacro"/>
   <!-- Parameters -->
   <xacro:property name="mass" value="10"/>
@@ -29,5 +30,5 @@
   <xacro:property name="visual_mesh_file" value="file://$(find desistek_saga_description)/mesh/saga.dae"/>
   <xacro:property name="collision_mesh_file" value="file://$(find desistek_saga_description)/mesh/saga.stl"/>
-  <xacro:macro name="desistek_saga_base" params="namespace debug">
+  <xacro:macro name="desistek_saga_base" params="namespace debug inertial_reference_frame">
   <link name="${namespace}/base_link">
     <inertial>
